Commit message: Step 18

File: body.urdf (robot description, URDF)
Before this commit: robot robot, 3 links, 2 joints
Joints:
- joint Torso_BackLeg: origin xyz=0 -1 1 rpy=0 0 0 -> xyz=0.5 0 1 rpy=0 0 0
- joint Torso_FrontLeg: origin xyz=0 1 1 rpy=0 0 0 -> xyz=-0.5 0 1 rpy=0 0 0

Commit message: Made body and legs

File: body.urdf (robot description, URDF)
Before this commit: robot robot, 9 links, 8 joints
Links:
- removed link BackLeg
- removed link BackLowerLeg
- removed link FrontLeg
- removed link FrontLowerLeg
- removed link LeftLeg
- removed link LeftLowerLeg
- removed link RightLeg
- removed link RightLowerLeg
- added link LeftFoot, mass 1; collision box size=0.25 0.5 0.05; visual box size=0.25 0.5 0.05
- added link LowerLeftLeg, mass 1; collision box size=0.25 0.25 0.7; visual box size=0.25 0.25 0.7
- added link LowerRightLeg, mass 1; collision box size=0.25 0.25 0.7; visual box size=0.25 0.25 0.7
- added link RightFoot, mass 1; collision box size=0.25 0.5 0.05; visual box size=0.25 0.5 0.05
- added link UpperLeftLeg, mass 1; collision box size=0.25 0.25 1; visual box size=0.25 0.25 1
- added link UpperRightLeg, mass 1; collision box size=0.25 0.25 1; visual box size=0.25 0.25 1
- link Torso: geometry collision box size=0.75 0.5 1; visual box size=0.75 0.5 1
Joints:
- removed joint BackLeg_BackLowerLeg
- removed joint FrontLeg_FrontLowerLeg
- removed joint LeftLeg_LeftLowerLeg
- removed joint RightLeg_RightLowerLeg
- removed joint Torso_BackLeg
- removed joint Torso_FrontLeg
- removed joint Torso_LeftLeg
- removed joint Torso_RightLeg
- added joint LowerLeftLeg_LeftFoot: type revolute, parent LowerLeftLeg, child LeftFoot, origin xyz=0 0 -0.7 rpy=0 0 0, axis 1 0 0, limit lower=-3.14159 upper=3.14159 effort=0.0 velocity=0.0
- added joint LowerRightLeg_RightFoot: type revolute, parent LowerRightLeg, child RightFoot, origin xyz=0 0 -0.7 rpy=0 0 0, axis 1 0 0, limit lower=-3.14159 upper=3.14159 effort=0.0 velocity=0.0
- added joint Torso_UpperLeftLeg: type revolute, parent Torso, child UpperLeftLeg, origin xyz=-0.375 0 1.75 rpy=0 0 0, axis 1 0 0, limit lower=-3.14159 upper=3.14159 effort=0.0 velocity=0.0
- added joint Torso_UpperRightLeg: type revolute, parent Torso, child UpperRightLeg, origin xyz=0.375 0 1.75 rpy=0 0 0, axis 1 0 0, limit lower=-3.14159 upper=3.14159 effort=0.0 velocity=0.0
- added joint UpperLeftLeg_LowerLeftLeg: type revolute, parent UpperLeftLeg, child LowerLeftLeg, origin xyz=-0.125 0 -1 rpy=0 0 0, axis 1 0 0, limit lower=-3.14159 upper=3.14159 effort=0.0 velocity=0.0
- added joint UpperRightLeg_LowerRightLeg: type revolute, parent UpperRightLeg, child LowerRightLeg, origin xyz=0.125 0 -1 rpy=0 0 0, axis 1 0 0, limit lower=-3.14159 upper=3.14159 effort=0.0 velocity=0.0

Commit message: Body complete

File: body.urdf (robot description, URDF)
Before this commit: robot robot, 7 links, 6 joints
Links:
- added link LowerLeftArm, mass 1; collision box size=0.25 0.7 0.25; visual box size=0.25 0.7 0.25
- added link LowerRightArm, mass 1; collision box size=0.25 0.7 0.25; visual box size=0.25 0.7 0.25
- added link UpperLeftArm, mass 1; collision box size=0.25 0.25 0.75; visual box size=0.25 0.25 0.75
- added link UpperRightArm, mass 1; collision box size=0.25 0.25 0.75; visual box size=0.25 0.25 0.75
- link Torso: geometry collision box size=0.75 0.5 1.5; visual box size=0.75 0.5 1.5
Joints:
- added joint Torso_UpperLeftArm: type revolute, parent Torso, child UpperLeftArm, origin xyz=-0.375 0 3.25 rpy=0 0 0, axis 1 0 0, limit lower=-3.14159 upper=3.14159 effort=0.0 velocity=0.0
- added joint Torso_UpperRightArm: type revolute, parent Torso, child UpperRightArm, origin xyz=0.375 0 3.25 rpy=0 0 0, axis 1 0 0, limit lower=-3.14159 upper=3.14159 effort=0.0 velocity=0.0
- added joint UpperLeftArm_LowerLeftArm: type revolute, parent UpperLeftArm, child LowerLeftArm, origin xyz=-0.125 0 -0.75 rpy=0 0 0, axis 1 0 0, limit lower=-3.14159 upper=3.14159 effort=0.0 velocity=0.0
- added joint UpperRightArm_LowerRightArm: type revolute, parent UpperRightArm, child LowerRightArm, origin xyz=0.125 0 -0.75 rpy=0 0 0, axis 1 0 0, limit lower=-3.14159 upper=3.14159 effort=0.0 velocity=0.0
- joint Torso_UpperLeftLeg: origin xyz=-0.375 0 1.75 rpy=0 0 0 -> xyz=-0.375 0 2 rpy=0 0 0
- joint Torso_UpperRightLeg: origin xyz=0.375 0 1.75 rpy=0 0 0 -> xyz=0.375 0 2 rpy=0 0 0

Commit message: Tests

File: body.urdf (robot description, URDF)
Before this commit: robot robot, 11 links, 10 joints
Links:
- removed link LeftFoot
- removed link LowerLeftArm
- removed link LowerLeftLeg
- removed link LowerRightArm
- removed link LowerRightLeg
- removed link RightFoot
- removed link UpperLeftArm
- removed link UpperLeftLeg
- removed link UpperRightArm
- removed link UpperRightLeg
- added link BackLeg, mass 1; collision box size=1 1 1; visual box size=1 1 1
- added link FrontLeg, mass 1; collision box size=1 1 1; visual box size=1 1 1
- link Torso: geometry collision box size=1 1 1; visual box size=1 1 1
Joints:
- removed joint LowerLeftLeg_LeftFoot
- removed joint LowerRightLeg_RightFoot
- removed joint Torso_UpperLeftArm
- removed joint Torso_UpperLeftLeg
- removed joint Torso_UpperRightArm
- removed joint Torso_UpperRightLeg
- removed joint UpperLeftArm_LowerLeftArm
- removed joint UpperLeftLeg_LowerLeftLeg
- removed joint UpperRightArm_LowerRightArm
- removed joint UpperRightLeg_LowerRightLeg
- added joint Torso_BackLeg: type revolute, parent Torso, child BackLeg, origin xyz=0.5 0 1 rpy=0 0 0, axis 0 1 0, limit lower=-3.14159 upper=3.14159 effort=0.0 velocity=0.0
- added joint Torso_FrontLeg: type revolute, parent Torso, child FrontLeg, origin xyz=-0.5 0 1 rpy=0 0 0, axis 0 1 0, limit lower=-3.14159 upper=3.14159 effort=0.0 velocity=0.0

Commit message: SOme more work

File: body.urdf (robot description, URDF)
Before this commit: robot robot, 3 links, 2 joints
Links:
- removed link BackLeg
- removed link FrontLeg
- added link LeftFoot, mass 1; collision box size=0.25 0.5 0.05; visual box size=0.25 0.5 0.05
- added link LowerLeftArm, mass 1; collision box size=0.25 0.7 0.25; visual box size=0.25 0.7 0.25
- added link LowerLeftLeg, mass 1; collision box size=0.25 0.25 0.95; visual box size=0.25 0.25 0.95
- added link LowerRightArm, mass 1; collision box size=0.25 0.7 0.25; visual box size=0.25 0.7 0.25
- added link LowerRightLeg, mass 1; collision box size=0.25 0.25 0.95; visual box size=0.25 0.25 0.95
- added link RightFoot, mass 1; collision box size=0.25 0.5 0.05; visual box size=0.25 0.5 0.05
- added link UpperLeftArm, mass 1; collision box size=0.25 0.25 0.75; visual box size=0.25 0.25 0.75
- added link UpperLeftLeg, mass 1; collision box size=0.25 0.25 1; visual box size=0.25 0.25 1
- added link UpperRightArm, mass 1; collision box size=0.25 0.25 0.75; visual box size=0.25 0.25 0.75
- added link UpperRightLeg, mass 1; collision box size=0.25 0.25 1; visual box size=0.25 0.25 1
- link Torso: geometry collision box size=0.75 0.5 1.5; visual box size=0.75 0.5 1.5
Joints:
- removed joint Torso_BackLeg
- removed joint Torso_FrontLeg
- added joint LowerLeftLeg_LeftFoot: type revolute, parent LowerLeftLeg, child LeftFoot, origin xyz=0 0 -0.95 rpy=0 0 0, axis 1 0 0, limit lower=-3.14159 upper=3.14159 effort=0.0 velocity=0.0
- added joint LowerRightLeg_RightFoot: type revolute, parent LowerRightLeg, child RightFoot, origin xyz=0 0 -0.95 rpy=0 0 0, axis 1 0 0, limit lower=-3.14159 upper=3.14159 effort=0.0 velocity=0.0
- added joint Torso_UpperLeftArm: type revolute, parent Torso, child UpperLeftArm, origin xyz=-0.375 0 3.25 rpy=0 0 0, axis 1 0 0, limit lower=-3.14159 upper=3.14159 effort=0.0 velocity=0.0
- added joint Torso_UpperLeftLeg: type revolute, parent Torso, child UpperLeftLeg, origin xyz=-0.375 0 2 rpy=0 0 0, axis 1 0 0, limit lower=-3.14159 upper=3.14159 effort=0.0 velocity=0.0
- added joint Torso_UpperRightArm: type revolute, parent Torso, child UpperRightArm, origin xyz=0.375 0 3.25 rpy=0 0 0, axis 1 0 0, limit lower=-3.14159 upper=3.14159 effort=0.0 velocity=0.0
- added joint Torso_UpperRightLeg: type revolute, parent Torso, child UpperRightLeg, origin xyz=0.375 0 2 rpy=0 0 0, axis 1 0 0, limit lower=-3.14159 upper=3.14159 effort=0.0 velocity=0.0
- added joint UpperLeftArm_LowerLeftArm: type revolute, parent UpperLeftArm, child LowerLeftArm, origin xyz=-0.125 0 -0.75 rpy=0 0 0, axis 1 0 0, limit lower=-3.14159 upper=3.14159 effort=0.0 velocity=0.0
- added joint UpperLeftLeg_LowerLeftLeg: type revolute, parent UpperLeftLeg, child LowerLeftLeg, origin xyz=-0.125 0 -1 rpy=0 0 0, axis 1 0 0, limit lower=-3.14159 upper=3.14159 effort=0.0 velocity=0.0
- added joint UpperRightArm_LowerRightArm: type revolute, parent UpperRightArm, child LowerRightArm, origin xyz=0.125 0 -0.75 rpy=0 0 0, axis 1 0 0, limit lower=-3.14159 upper=3.14159 effort=0.0 velocity=0.0
- added joint UpperRightLeg_LowerRightLeg: type revolute, parent UpperRightLeg, child LowerRightLeg, origin xyz=0.125 0 -1 rpy=0 0 0, axis 1 0 0, limit lower=-3.14159 upper=3.14159 effort=0.0 velocity=0.0
