Commit message: Random Shapes

File: body0.urdf (robot description, URDF)
Before this commit: robot robot, 3 links, 2 joints
Links:
- removed link Part0
- added link Part2, mass 1; collision box size=2.0 2.5 1; visual box size=2.0 2.5 1
- added link Part3, mass 1; collision box size=2.5 3.5 1; visual box size=2.5 3.5 1
- link Part1: geometry collision box size=1.5 1.5 1; visual box size=1.5 1.5 1
Joints:
- removed joint Part0_Part1
- removed joint Torso_Part0
- added joint Part1_Part2: type revolute, parent Part1, child Part2, origin xyz=0 1.5 0 rpy=0 0 0, axis 1 0 0, limit lower=-3.14159 upper=3.14159 effort=0.0 velocity=0.0
- added joint Part2_Part3: type revolute, parent Part2, child Part3, origin xyz=0 2.5 0 rpy=0 0 0, axis 1 0 0, limit lower=-3.14159 upper=3.14159 effort=0.0 velocity=0.0
- added joint Torso_Part1: type revolute, parent Torso, child Part1, origin xyz=0 0.5 0.5 rpy=0 0 0, axis 1 0 0, limit lower=-3.14159 upper=3.14159 effort=0.0 velocity=0.0

Commit message: Random Snake - Complete

File: body0.urdf (robot description, URDF)
Before this commit: robot robot, 4 links, 3 joints
Links:
- removed link Torso
- added link Part0, mass 1; collision box size=0.88 0.88 0.88; visual box size=0.88 0.88 0.88
- added link Part4, mass 1; collision box size=0.53 0.53 0.53; visual box size=0.53 0.53 0.53
- added link Part5, mass 1; collision box size=0.98 0.98 0.98; visual box size=0.98 0.98 0.98
- added link Part6, mass 1; collision box size=0.53 0.53 0.53; visual box size=0.53 0.53 0.53
- link Part1: geometry collision box size=0.54 0.54 0.54; visual box size=0.54 0.54 0.54
- link Part2: geometry collision box size=0.76 0.76 0.76; visual box size=0.76 0.76 0.76
- link Part3: geometry collision box size=0.99 0.99 0.99; visual box size=0.99 0.99 0.99
Joints:
- removed joint Torso_Part1
- added joint Part0_Part1: type revolute, parent Part0, child Part1, origin xyz=0 0.44 0.5 rpy=0 0 0, axis 1 0 0, limit lower=-3.14159 upper=3.14159 effort=0.0 velocity=0.0
- added joint Part3_Part4: type revolute, parent Part3, child Part4, origin xyz=0 0.99 0 rpy=0 0 0, axis 1 0 0, limit lower=-3.14159 upper=3.14159 effort=0.0 velocity=0.0
- added joint Part4_Part5: type revolute, parent Part4, child Part5, origin xyz=0 0.53 0 rpy=0 0 0, axis 1 0 0, limit lower=-3.14159 upper=3.14159 effort=0.0 velocity=0.0
- added joint Part5_Part6: type revolute, parent Part5, child Part6, origin xyz=0 0.98 0 rpy=0 0 0, axis 1 0 0, limit lower=-3.14159 upper=3.14159 effort=0.0 velocity=0.0
- joint Part1_Part2: origin xyz=0 1.5 0 rpy=0 0 0 -> xyz=0 0.54 0 rpy=0 0 0
- joint Part2_Part3: origin xyz=0 2.5 0 rpy=0 0 0 -> xyz=0 0.76 0 rpy=0 0 0
