Commit message: No Bias Random PHC

File: results/body31.urdf (robot description, URDF)
Before this commit: robot robot, 4 links, 3 joints
Links:
- link Part0: geometry collision box size=0.38 0.3 0.98; visual box size=0.38 0.3 0.98
- link Part1: geometry collision box size=0.67 0.89 0.48; visual box size=0.67 0.89 0.48
- link Part2: geometry collision box size=0.4 0.28 0.62; visual box size=0.4 0.28 0.62
- link Part3: geometry collision box size=0.97 0.92 0.44; visual box size=0.97 0.92 0.44
Joints:
- removed joint Part1_Part3
- added joint Part2_Part3: type revolute, parent Part2, child Part3, origin xyz=0.2 0.0 0.31 rpy=0 0 0, axis 0 0 1, limit lower=-3.14159 upper=3.14159 effort=0.0 velocity=0.0
- joint Part0_Part1: axis 1 0 0 -> 0 1 0; origin xyz=0.0 0.0 0.54 rpy=0 0 0 -> xyz=0.0 0.15 0.49 rpy=0 0 0
- joint Part1_Part2: axis 0 1 0 -> 1 0 0; origin xyz=0.0 0.435 0.425 rpy=0 0 0 -> xyz=0.335 0.445 0.0 rpy=0 0 0

File: results/evolved/4673/body4673.urdf (robot description, URDF)
Before this commit: robot robot, 10 links, 9 joints
Links:
- link Part0: geometry collision box size=0.74 0.45 0.26; visual box size=0.74 0.45 0.26
- link Part1: geometry collision box size=0.72 0.6 0.91; visual box size=0.72 0.6 0.91
- link Part2: geometry collision box size=0.81 0.97 0.96; visual box size=0.81 0.97 0.96
- link Part3: geometry collision box size=0.49 0.68 0.4; visual box size=0.49 0.68 0.4
- link Part4: geometry collision box size=0.95 0.85 0.58; visual box size=0.95 0.85 0.58
- link Part5: geometry collision box size=0.47 0.83 0.99; visual box size=0.47 0.83 0.99
- link Part6: geometry collision box size=0.44 0.88 0.75; visual box size=0.44 0.88 0.75
- link Part7: geometry collision box size=0.86 0.72 0.61; visual box size=0.86 0.72 0.61
- link Part8: geometry collision box size=0.83 0.34 0.34; visual box size=0.83 0.34 0.34
- link Part9: geometry collision box size=0.72 0.88 0.36; visual box size=0.72 0.88 0.36
Joints:
- removed joint Part2_Part3
- removed joint Part4_Part6
- removed joint Part4_Part7
- removed joint Part8_Part9
- added joint Part1_Part3: type revolute, parent Part1, child Part3, origin xyz=0.0 0.3 -0.455 rpy=0 0 0, axis 1 0 0, limit lower=-3.14159 upper=3.14159 effort=0.0 velocity=0.0
- added joint Part1_Part7: type revolute, parent Part1, child Part7, origin xyz=0.0 0.0 -0.91 rpy=0 0 0, axis 1 0 0, limit lower=-3.14159 upper=3.14159 effort=0.0 velocity=0.0
- added joint Part2_Part9: type revolute, parent Part2, child Part9, origin xyz=-0.405 -0.485 0.0 rpy=0 0 0, axis 0 0 1, limit lower=-3.14159 upper=3.14159 effort=0.0 velocity=0.0
- added joint Part3_Part6: type revolute, parent Part3, child Part6, origin xyz=0.0 0.68 0.0 rpy=0 0 0, axis 0 0 1, limit lower=-3.14159 upper=3.14159 effort=0.0 velocity=0.0
- joint Part0_Part1: axis 1 0 0 -> 0 0 1; origin xyz=0.0 0.245 0.5 rpy=0 0 0 -> xyz=0.0 0.0 1.52 rpy=0 0 0
- joint Part1_Part2: axis 0 1 0 -> 1 0 0; origin xyz=0.0 0.415 0.5 rpy=0 0 0 -> xyz=-0.36 0.0 -0.455 rpy=0 0 0
- joint Part2_Part4: axis 0 1 0 -> 1 0 0; origin xyz=0.0 0.485 0.42 rpy=0 0 0 -> xyz=-0.405 0.0 0.48 rpy=0 0 0
- joint Part2_Part5: axis 1 0 0 -> 0 0 1; origin xyz=-0.15 0.0 0.42 rpy=0 0 0 -> xyz=-0.405 0.0 0.48 rpy=0 0 0
- joint Part4_Part8: axis 1 0 0 -> 0 0 1; origin xyz=0.0 0.21 0.4 rpy=0 0 0 -> xyz=0.475 0.0 0.29 rpy=0 0 0
