Commit message: Mid Work

File: results/body33.urdf (robot description, URDF)
Before this commit: robot robot, 4 links, 3 joints
Links:
- link Part0: geometry collision box size=0.62 0.69 0.41; visual box size=0.62 0.69 0.41
- link Part1: geometry collision box size=0.4 0.76 0.63; visual box size=0.4 0.76 0.63
- link Part2: geometry collision box size=0.73 0.35 0.7; visual box size=0.73 0.35 0.7
- link Part3: geometry collision box size=0.97 0.89 0.43; visual box size=0.97 0.89 0.43
Joints:
- removed joint Part2_Part3
- added joint Part1_Part3: type revolute, parent Part1, child Part3, origin xyz=0.0 0.38 0.315 rpy=0 0 0, axis 1 0 0, limit lower=-3.14159 upper=3.14159 effort=0.0 velocity=0.0
- joint Part0_Part1: axis 0 1 0 -> 1 0 0; origin xyz=0.0 0.15 0.49 rpy=0 0 0 -> xyz=0.0 0.0 0.4099999999999999 rpy=0 0 0
- joint Part1_Part2: axis 1 0 0 -> 0 0 1; origin xyz=0.335 0.445 0.0 rpy=0 0 0 -> xyz=0.2 0.0 0.315 rpy=0 0 0

File: results/body8.urdf (robot description, URDF)
Before this commit: robot robot, 2 links, 1 joints
Links:
- link Part0: geometry collision box size=0.79 0.74 0.98; visual box size=0.79 0.74 0.98
- link Part1: geometry collision box size=0.89 0.82 0.46; visual box size=0.89 0.82 0.46
Joints:
- joint Part0_Part1: axis 1 0 0 -> 0 1 0; origin xyz=0.0 -0.23 0.47 rpy=0 0 0 -> xyz=0.395 0.0 0.49 rpy=0 0 0
