Commit message: Cleanup

File: results/body0.urdf (robot description, URDF)
Before this commit: robot robot, 4 links, 3 joints
Links:
- link Part0: geometry collision box size=0.29 0.74 0.38; visual box size=0.29 0.74 0.38
- link Part1: geometry collision box size=0.29 0.33 0.96; visual box size=0.29 0.33 0.96
- link Part2: geometry collision box size=0.26 0.7 0.88; visual box size=0.26 0.7 0.88
- link Part3: geometry collision box size=0.46 0.97 0.9; visual box size=0.46 0.97 0.9
Joints:
- removed joint Part1_Part2
- removed joint Part1_Part3
- added joint Part0_Part2: type revolute, parent Part0, child Part2, origin xyz=-0.145 0.0 0.45 rpy=0 0 0, axis 0 0 1, limit lower=-3.14159 upper=3.14159 effort=0.0 velocity=0.0
- added joint Part2_Part3: type revolute, parent Part2, child Part3, origin xyz=-0.13 0.35 0.0 rpy=0 0 0, axis 1 0 0, limit lower=-3.14159 upper=3.14159 effort=0.0 velocity=0.0
- joint Part0_Part1: origin xyz=0.0 0.0 0.4099999999999999 rpy=0 0 0 -> xyz=0.0 0.0 0.6399999999999999 rpy=0 0 0

Commit message: Testing

File: results/body0.urdf (robot description, URDF)
Before this commit: robot robot, 4 links, 3 joints
Links:
- added link Part4, mass 1; collision box size=0.52 0.79 0.28; visual box size=0.52 0.79 0.28
- added link Part5, mass 1; collision box size=0.88 0.95 0.54; visual box size=0.88 0.95 0.54
- added link Part6, mass 1; collision box size=0.53 0.83 0.62; visual box size=0.53 0.83 0.62
- link Part0: geometry collision box size=0.4 0.88 0.82; visual box size=0.4 0.88 0.82
- link Part1: geometry collision box size=0.87 0.28 0.74; visual box size=0.87 0.28 0.74
- link Part2: geometry collision box size=0.82 0.59 0.54; visual box size=0.82 0.59 0.54
- link Part3: geometry collision box size=0.28 0.27 0.28; visual box size=0.28 0.27 0.28
Joints:
- removed joint Part2_Part3
- added joint Part1_Part3: type revolute, parent Part1, child Part3, origin xyz=-0.435 0.0 -0.37 rpy=0 0 0, axis 1 0 0, limit lower=-3.14159 upper=3.14159 effort=0.0 velocity=0.0
- added joint Part3_Part4: type revolute, parent Part3, child Part4, origin xyz=0.0 0.0 -0.28 rpy=0 0 0, axis 1 0 0, limit lower=-3.14159 upper=3.14159 effort=0.0 velocity=0.0
- added joint Part3_Part5: type revolute, parent Part3, child Part5, origin xyz=-0.14 0.0 -0.14 rpy=0 0 0, axis 1 0 0, limit lower=-3.14159 upper=3.14159 effort=0.0 velocity=0.0
- added joint Part5_Part6: type revolute, parent Part5, child Part6, origin xyz=-0.44 0.475 0.0 rpy=0 0 0, axis 0 1 0, limit lower=-3.14159 upper=3.14159 effort=0.0 velocity=0.0
- joint Part0_Part1: axis 1 0 0 -> 0 0 1; origin xyz=0.0 0.0 0.6399999999999999 rpy=0 0 0 -> xyz=-0.2 0.0 0.93 rpy=0 0 0
- joint Part0_Part2: axis 0 0 1 -> 1 0 0; origin xyz=-0.145 0.0 0.45 rpy=0 0 0 -> xyz=0.0 -0.44 0.93 rpy=0 0 0
