Commit message: Progress

File: results/body3929.urdf (robot description, URDF)
Before this commit: robot robot, 10 links, 9 joints
Links:
- added link Part10, mass 1; collision box size=0.94 0.62 0.42; visual box size=0.94 0.62 0.42
- link Part0: geometry collision box size=0.35 0.42 0.35; visual box size=0.35 0.42 0.35
- link Part1: geometry collision box size=0.46 0.66 0.81; visual box size=0.46 0.66 0.81
- link Part2: geometry collision box size=0.52 0.4 0.8; visual box size=0.52 0.4 0.8
- link Part3: geometry collision box size=0.4 0.62 0.6; visual box size=0.4 0.62 0.6
- link Part4: geometry collision box size=0.49 0.92 0.81; visual box size=0.49 0.92 0.81
- link Part5: geometry collision box size=0.56 0.58 0.51; visual box size=0.56 0.58 0.51
- link Part6: geometry collision box size=0.5 0.59 0.64; visual box size=0.5 0.59 0.64
- link Part7: geometry collision box size=0.82 0.46 0.94; visual box size=0.82 0.46 0.94
- link Part8: geometry collision box size=0.4 0.51 0.98; visual box size=0.4 0.51 0.98
- link Part9: geometry collision box size=0.38 0.28 0.4; visual box size=0.38 0.28 0.4
Joints:
- removed joint Part1_Part7
- removed joint Part2_Part4
- removed joint Part2_Part5
- removed joint Part2_Part9
- removed joint Part3_Part6
- removed joint Part4_Part8
- added joint Part0_Part10: type revolute, parent Part0, child Part10, origin xyz=0.175 0.0 1.215 rpy=0 0 0, axis 0 0 1, limit lower=-3.14159 upper=3.14159 effort=0.0 velocity=0.0
- added joint Part0_Part4: type revolute, parent Part0, child Part4, origin xyz=0.0 -0.21 1.215 rpy=0 0 0, axis 1 0 0, limit lower=-3.14159 upper=3.14159 effort=0.0 velocity=0.0
- added joint Part0_Part5: type revolute, parent Part0, child Part5, origin xyz=-0.175 0.0 1.215 rpy=0 0 0, axis 1 0 0, limit lower=-3.14159 upper=3.14159 effort=0.0 velocity=0.0
- added joint Part4_Part6: type revolute, parent Part4, child Part6, origin xyz=0.0 -0.46 -0.405 rpy=0 0 0, axis 0 1 0, limit lower=-3.14159 upper=3.14159 effort=0.0 velocity=0.0
- added joint Part4_Part9: type revolute, parent Part4, child Part9, origin xyz=0.0 -0.46 -0.405 rpy=0 0 0, axis 0 0 1, limit lower=-3.14159 upper=3.14159 effort=0.0 velocity=0.0
- added joint Part6_Part7: type revolute, parent Part6, child Part7, origin xyz=-0.25 0.0 -0.32 rpy=0 0 0, axis 0 1 0, limit lower=-3.14159 upper=3.14159 effort=0.0 velocity=0.0
- added joint Part6_Part8: type revolute, parent Part6, child Part8, origin xyz=0.0 -0.295 -0.32 rpy=0 0 0, axis 1 0 0, limit lower=-3.14159 upper=3.14159 effort=0.0 velocity=0.0
- joint Part0_Part1: origin xyz=0.0 0.0 1.52 rpy=0 0 0 -> xyz=0.0 0.21 1.215 rpy=0 0 0
- joint Part1_Part2: axis 1 0 0 -> 0 0 1; origin xyz=-0.36 0.0 -0.455 rpy=0 0 0 -> xyz=0.0 0.33 -0.405 rpy=0 0 0
- joint Part1_Part3: axis 1 0 0 -> 0 1 0; origin xyz=0.0 0.3 -0.455 rpy=0 0 0 -> xyz=0.0 0.66 0.0 rpy=0 0 0
