Commit message: First Good Run

File: results/asym/4230/body4230.urdf (robot description, URDF)
Before this commit: robot robot, 11 links, 10 joints
Links:
- added link Part11, mass 1; collision box size=0.26 0.75 0.75; visual box size=0.26 0.75 0.75
- link Part0: geometry collision box size=0.86 0.98 0.26; visual box size=0.86 0.98 0.26
- link Part1: geometry collision box size=0.87 0.6 0.45; visual box size=0.87 0.6 0.45
- link Part10: geometry collision box size=0.85 0.63 0.29; visual box size=0.85 0.63 0.29
- link Part2: geometry collision box size=0.46 0.64 0.53; visual box size=0.46 0.64 0.53
- link Part3: geometry collision box size=0.97 0.71 0.48; visual box size=0.97 0.71 0.48
- link Part4: geometry collision box size=1.0 0.46 0.34; visual box size=1.0 0.46 0.34
- link Part5: geometry collision box size=0.28 0.7 0.56; visual box size=0.28 0.7 0.56
- link Part6: geometry collision box size=0.49 0.52 0.88; visual box size=0.49 0.52 0.88
- link Part7: geometry collision box size=0.87 0.92 0.55; visual box size=0.87 0.92 0.55
- link Part8: geometry collision box size=0.66 0.3 0.46; visual box size=0.66 0.3 0.46
- link Part9: geometry collision box size=0.86 0.89 0.79; visual box size=0.86 0.89 0.79
Joints:
- removed joint Part0_Part10
- removed joint Part0_Part4
- removed joint Part0_Part5
- removed joint Part1_Part2
- removed joint Part1_Part3
- removed joint Part4_Part6
- removed joint Part4_Part9
- removed joint Part6_Part7
- removed joint Part6_Part8
- added joint Part0_Part2: type revolute, parent Part0, child Part2, origin xyz=0.0 0.0 1.32 rpy=0 0 0, axis 1 0 0, limit lower=-3.14159 upper=3.14159 effort=0.0 velocity=0.0
- added joint Part0_Part3: type revolute, parent Part0, child Part3, origin xyz=0.0 0.49 1.4500000000000002 rpy=0 0 0, axis 1 0 0, limit lower=-3.14159 upper=3.14159 effort=0.0 velocity=0.0
- added joint Part1_Part5: type revolute, parent Part1, child Part5, origin xyz=0.87 0.0 0.0 rpy=0 0 0, axis 1 0 0, limit lower=-3.14159 upper=3.14159 effort=0.0 velocity=0.0
- added joint Part2_Part9: type revolute, parent Part2, child Part9, origin xyz=0.0 0.0 -0.53 rpy=0 0 0, axis 0 1 0, limit lower=-3.14159 upper=3.14159 effort=0.0 velocity=0.0
- added joint Part3_Part4: type revolute, parent Part3, child Part4, origin xyz=-0.485 0.355 0.0 rpy=0 0 0, axis 0 0 1, limit lower=-3.14159 upper=3.14159 effort=0.0 velocity=0.0
- added joint Part3_Part6: type revolute, parent Part3, child Part6, origin xyz=0.0 0.71 0.0 rpy=0 0 0, axis 0 1 0, limit lower=-3.14159 upper=3.14159 effort=0.0 velocity=0.0
- added joint Part4_Part7: type revolute, parent Part4, child Part7, origin xyz=-1.0 0.0 0.0 rpy=0 0 0, axis 0 0 1, limit lower=-3.14159 upper=3.14159 effort=0.0 velocity=0.0
- added joint Part4_Part8: type revolute, parent Part4, child Part8, origin xyz=-0.5 -0.23 0.0 rpy=0 0 0, axis 0 1 0, limit lower=-3.14159 upper=3.14159 effort=0.0 velocity=0.0
- added joint Part7_Part10: type revolute, parent Part7, child Part10, origin xyz=-0.435 -0.46 0.0 rpy=0 0 0, axis 0 1 0, limit lower=-3.14159 upper=3.14159 effort=0.0 velocity=0.0
- added joint Part7_Part11: type revolute, parent Part7, child Part11, origin xyz=-0.435 0.0 0.275 rpy=0 0 0, axis 0 0 1, limit lower=-3.14159 upper=3.14159 effort=0.0 velocity=0.0
- joint Part0_Part1: origin xyz=0.0 0.21 1.215 rpy=0 0 0 -> xyz=0.43 0.0 1.4500000000000002 rpy=0 0 0
